File: PCB/Displays_Strip/lcd.kicad_sch (KiCad schematic)
At the start: 16 parts, among them U10 DT010ATFT, U11 DT010ATFT, U12 CAT4104V-GT3, U13 CAT4104V-GT3, U14 CAT4104V-GT3, U2 DT010ATFT, U3 DT010ATFT, U4 DT010ATFT, U5 DT010ATFT, U6 DT010ATFT, U7 DT010ATFT, U8 DT010ATFT, U9 DT010ATFT

Commit message: Schematic Flash
Parts:
- U10, U11, U2, U3, U4, U5, U6, U7, U8, U9: footprint (none) -> Console:Hirose FFC FPC 13 Pin Inverted
Changed lines of the file:
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@@
 			)
 		)
-		(property "Footprint" ""
+		(property "Footprint" "Console:Hirose FFC FPC 13 Pin Inverted"
 			(at 129.54 93.98 0)
 			(effects
@@
 			)
 		)
-		(property "Footprint" ""
+		(property "Footprint" "Console:Hirose FFC FPC 13 Pin Inverted"
 			(at 53.34 129.54 0)
 			(effects
@@
 			)
 		)
-		(property "Footprint" ""
+		(property "Footprint" "Console:Hirose FFC FPC 13 Pin Inverted"
 			(at 129.54 129.54 0)
 			(effects
@@
 			)
 		)
-		(property "Footprint" ""
+		(property "Footprint" "Console:Hirose FFC FPC 13 Pin Inverted"
 			(at 53.34 93.98 0)
 			(effects
@@
 			)
 		)
-		(property "Footprint" ""
+		(property "Footprint" "Console:Hirose FFC FPC 13 Pin Inverted"
 			(at 129.54 58.42 0)
 			(effects
@@
 			)
 		)
-		(property "Footprint" ""
+		(property "Footprint" "Console:Hirose FFC FPC 13 Pin Inverted"
 			(at 129.54 165.1 0)
 			(effects
@@
 			)
 		)
-		(property "Footprint" ""
+		(property "Footprint" "Console:Hirose FFC FPC 13 Pin Inverted"
 			(at 53.34 58.42 0)
 			(effects
@@
 			)
 		)
-		(property "Footprint" ""
+		(property "Footprint" "Console:Hirose FFC FPC 13 Pin Inverted"
 			(at 129.54 22.86 0)
 			(effects
@@
 			)
 		)
-		(property "Footprint" ""
+		(property "Footprint" "Console:Hirose FFC FPC 13 Pin Inverted"
 			(at 53.34 165.1 0)
 			(effects
@@
 			)
 		)
-		(property "Footprint" ""
+		(property "Footprint" "Console:Hirose FFC FPC 13 Pin Inverted"
 			(at 53.34 22.86 0)
 			(effects
