File: PCB/Buttons_Flash/Matrix.kicad_sch (KiCad schematic)
At the start: 60 parts

Commit message: PCB Buttons Flash
Connections:
- net at SW1.0: now also D1.2 (A)
- net at SW6.0: now also D6.2 (A)
- net at SW13.0: now also D13.2 (A)
- net at SW8.0: now also D8.2 (A)
- net at SW11.0: now also D11.2 (A)
- net at SW5.0: now also D5.2 (A)
- net at SW19.0: now also D19.2 (A)
- net at SW15.0: now also D15.2 (A)
Changed lines of the file:
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@@
 	)
 	(symbol
-		(lib_name "Console:Digitast")
 		(lib_id "Console:Digitast")
 		(at 55.88 57.15 0)
@@
 	)
 	(symbol
-		(lib_name "Console:Digitast")
 		(lib_id "Console:Digitast")
 		(at 195.58 57.15 0)
@@
 	)
 	(symbol
-		(lib_name "Console:Digitast")
 		(lib_id "Console:Digitast")
 		(at 167.64 82.55 0)
@@
 	)
 	(symbol
-		(lib_name "Console:Digitast")
 		(lib_id "Console:Digitast")
 		(at 195.58 82.55 0)
@@
 	)
 	(symbol
-		(lib_name "Console:Digitast")
 		(lib_id "Console:Digitast")
 		(at 251.46 57.15 0)
@@
 	)
 	(symbol
-		(lib_name "Console:Digitast")
 		(lib_id "Console:Digitast")
 		(at 251.46 82.55 0)
@@
 	)
 	(symbol
-		(lib_name "Console:Digitast")
 		(lib_id "Console:Digitast")
 		(at 223.52 57.15 0)
@@
 	)
 	(symbol
-		(lib_name "Console:Digitast")
 		(lib_id "Console:Digitast")
 		(at 111.76 82.55 0)
@@
 	)
 	(symbol
-		(lib_name "Console:Digitast")
 		(lib_id "Console:Digitast")
 		(at 55.88 82.55 0)
@@
 	)
 	(symbol
-		(lib_name "Console:Digitast")
 		(lib_id "Console:Digitast")
 		(at 83.82 82.55 0)
@@
 	)
 	(symbol
-		(lib_name "Console:Digitast")
 		(lib_id "Console:Digitast")
 		(at 55.88 107.95 0)
@@
 	)
 	(symbol
-		(lib_name "Console:Digitast")
 		(lib_id "Console:Digitast")
 		(at 167.64 57.15 0)
@@
 	)
 	(symbol
-		(lib_name "Console:Digitast")
 		(lib_id "Console:Digitast")
 		(at 83.82 57.15 0)
@@
 	)
 	(symbol
-		(lib_name "Console:Digitast")
 		(lib_id "Console:Digitast")
 		(at 111.76 107.95 0)
@@
 	)
 	(symbol
-		(lib_name "Console:Digitast")
 		(lib_id "Console:Digitast")
 		(at 139.7 107.95 0)
@@
 	)
 	(symbol
-		(lib_name "Console:Digitast")
 		(lib_id "Console:Digitast")
 		(at 223.52 82.55 0)
@@
 	)
 	(symbol
-		(lib_name "Console:Digitast")
 		(lib_id "Console:Digitast")
 		(at 111.76 57.15 0)
@@
 	)
 	(symbol
-		(lib_name "Console:Digitast")
 		(lib_id "Console:Digitast")
 		(at 83.82 107.95 0)
@@
 	)
 	(symbol
-		(lib_name "Console:Digitast")
 		(lib_id "Console:Digitast")
 		(at 139.7 57.15 0)
@@
 	)
 	(symbol
-		(lib_name "Console:Digitast")
 		(lib_id "Console:Digitast")
 		(at 139.7 82.55 0)
