File: PCB/Buttons_Flash/Buttons_Flash.kicad_pcb (KiCad board)
At the start: 2 copper layers, 80 parts, among them J1 Switches, J2 LEDs, J3 Power, U1 74HC595, U2 74HC595, U3 74HC595, U4 74HC165

Commit message: PCB Buttons Flash
Parts:
- added H1: MountingHole, MountingHole:MountingHole_3.2mm_M3, F.Cu at (25.0, 87.0)
- added H2: MountingHole, MountingHole:MountingHole_3.2mm_M3, F.Cu at (145.5, 87.0)
- added H3: MountingHole, MountingHole:MountingHole_3.2mm_M3, F.Cu at (270.0, 87.0)
- added H4: MountingHole, MountingHole:MountingHole_3.2mm_M3, F.Cu at (25.0, 145.0)
- added H5: MountingHole, MountingHole:MountingHole_3.2mm_M3, F.Cu at (145.5, 145.0)
- added H6: MountingHole, MountingHole:MountingHole_3.2mm_M3, F.Cu at (270.0, 145.0)
- moved D10 307.1 mm to (65.5, 127.0), turned to 180 degrees
- moved SW10 305.5 mm to (57.0, 127.0)
- moved R10 303.2 mm to (49.0, 118.5)
- moved D9 290.0 mm to (40.5, 127.0), turned to 180 degrees
- moved SW9 288.3 mm to (32.0, 127.0)
- moved R9 286.1 mm to (24.0, 118.5)
- moved J1 255.9 mm to (271.0, 136.5), turned to 180 degrees
- moved C3 248.9 mm to (256.5, 144.5), turned to 0 degrees
- moved U3 234.8 mm to (249.0, 142.0), turned to -90 degrees
- moved J3 225.8 mm to (271.0, 117.8), turned to 180 degrees
- moved C5 220.2 mm to (267.0, 116.5), turned to 90 degrees
- moved C4 218.9 mm to (241.0, 143.5), turned to 90 degrees
- moved J2 211.1 mm to (271.0, 109.3), turned to 180 degrees
- moved U4 206.6 mm to (234.5, 142.0), turned to -90 degrees
- moved U2 179.9 mm to (253.1, 88.8)
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Routing:
- net /Matrix/SW_C0: track 0.00 -> 294.4 mm, vias 0 -> 6
- net /Matrix/SW_R0: track 0.00 -> 279.7 mm, vias 0 -> 1
- net /Matrix/SW_C1: track 0.00 -> 278.6 mm, vias 0 -> 6
- net /Matrix/LED_C0: track 0.00 -> 253.6 mm, vias 0 -> 2
- net /Matrix/SW_R1: track 0.00 -> 247.2 mm, vias 0 -> 1
- net /Matrix/LED_R1: track 0.00 -> 243.7 mm, vias 0 -> 4
- net /Matrix/LED_C1: track 0.00 -> 238.0 mm, vias 0 -> 2
- net /Matrix/LED_R0: track 0.00 -> 232.2 mm, vias 0 -> 2
- net /Matrix/LED_C2: track 0.00 -> 230.1 mm, vias 0 -> 4
- net /Matrix/LED_C3: track 0.00 -> 224.7 mm, vias 0 -> 3
- net /Matrix/SW_C2: track 0.00 -> 207.6 mm, vias 0 -> 4
- net /Matrix/SW_C3: track 0.00 -> 207.6 mm, vias 0 -> 4
- net +3.3V: track 0.00 -> 155.7 mm
- net /Matrix/LED_C4: track 0.00 -> 132.3 mm, vias 0 -> 1
- net /Matrix/SW_C4: track 0.00 -> 126.4 mm, vias 0 -> 2
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- added copper zone on B.Cu, net GND
- added copper zone on F.Cu, net GND
Other:
- board outline added: 255 x 68 mm
- board text added: "1"
- board text added: "3.3"
- board text added: "Console v2.0 Flash Buttons v1.0 C. Güse"
- board text added: "GND"
- board text added: "LEDs"
- board text added: "Switches"

Commit message: Fader Breakout Board
Changed lines of the file:
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@@
 			(plot_on_all_layers_selection 0x0000000_00000000)
 			(disableapertmacros no)
-			(usegerberextensions no)
-			(usegerberattributes yes)
-			(usegerberadvancedattributes yes)
-			(creategerberjobfile yes)
+			(usegerberextensions yes)
+			(usegerberattributes no)
+			(usegerberadvancedattributes no)
+			(creategerberjobfile no)
 			(dashed_line_dash_ratio 12.000000)
 			(dashed_line_gap_ratio 3.000000)
@@
 			(psa4output no)
 			(plotreference yes)
-			(plotvalue yes)
+			(plotvalue no)
 			(plotfptext yes)
 			(plotinvisibletext no)
 			(sketchpadsonfab no)
-			(subtractmaskfromsilk no)
+			(subtractmaskfromsilk yes)
 			(outputformat 1)
 			(mirror no)
@@
 				(font
 					(size 1 1)
-					(thickness 0.1)
+					(thickness 0.15)
 				)
 			)
@@
 			(size 1.1176 1.1176)
 			(drill 1.1176)
-			(layers "F&B.Cu" "*.Mask")
+			(layers "*.Cu" "*.Mask")
 		)
 		(pad "" np_thru_hole circle
@@
 			(size 1.1176 1.1176)
 			(drill 1.1176)
-			(layers "F&B.Cu" "*.Mask")
+			(layers "*.Cu" "*.Mask")
 		)
 		(pad "+" thru_hole oval
@@
 				(font
 					(size 1 1)
-					(thickness 0.1)
+					(thickness 0.15)
 				)
 			)
@@
 			(size 1.1176 1.1176)
 			(drill 1.1176)
-			(layers "F&B.Cu" "*.Mask")
+			(layers "*.Cu" "*.Mask")
 		)
 		(pad "" np_thru_hole circle
@@
 			(size 1.1176 1.1176)
 			(drill 1.1176)
-			(layers "F&B.Cu" "*.Mask")
+			(layers "*.Cu" "*.Mask")
 		)
 		(pad "+" thru_hole oval
@@
 				(font
 					(size 1 1)
-					(thickness 0.1)
+					(thickness 0.15)
 				)
 			)
@@
 			(size 1.1176 1.1176)
 			(drill 1.1176)
-			(layers "F&B.Cu" "*.Mask")
+			(layers "*.Cu" "*.Mask")
 		)
 		(pad "" np_thru_hole circle
@@
 			(size 1.1176 1.1176)
 			(drill 1.1176)
-			(layers "F&B.Cu" "*.Mask")
+			(layers "*.Cu" "*.Mask")
 		)
 		(pad "+" thru_hole oval
@@
 				(font
 					(size 1 1)
-					(thickness 0.1)
+					(thickness 0.15)
 				)
 			)
@@
 			(size 1.1176 1.1176)
 			(drill 1.1176)
-			(layers "F&B.Cu" "*.Mask")
+			(layers "*.Cu" "*.Mask")
 		)
 		(pad "" np_thru_hole circle
@@
 			(size 1.1176 1.1176)
 			(drill 1.1176)
-			(layers "F&B.Cu" "*.Mask")
+			(layers "*.Cu" "*.Mask")
 		)
 		(pad "+" thru_hole oval
@@
 				(font
 					(size 1 1)
-					(thickness 0.1)
+					(thickness 0.15)
 				)
 			)
@@
 			(size 1.1176 1.1176)
 			(drill 1.1176)
-			(layers "F&B.Cu" "*.Mask")
+			(layers "*.Cu" "*.Mask")
 		)
 		(pad "" np_thru_hole circle
@@
 			(size 1.1176 1.1176)
 			(drill 1.1176)
-			(layers "F&B.Cu" "*.Mask")
+			(layers "*.Cu" "*.Mask")
 		)
 		(pad "+" thru_hole oval
@@
 				(font
 					(size 1 1)
-					(thickness 0.1)
+					(thickness 0.15)
 				)
 			)
@@
 			(size 1.1176 1.1176)
 			(drill 1.1176)
-			(layers "F&B.Cu" "*.Mask")
+			(layers "*.Cu" "*.Mask")
 		)
 		(pad "" np_thru_hole circle
@@
 			(size 1.1176 1.1176)
 			(drill 1.1176)
-			(layers "F&B.Cu" "*.Mask")
+			(layers "*.Cu" "*.Mask")
 		)
 		(pad "+" thru_hole oval
@@
 				(font
 					(size 1 1)
-					(thickness 0.1)
+					(thickness 0.15)
 				)
 			)
@@
 			(size 1.1176 1.1176)
 			(drill 1.1176)
-			(layers "F&B.Cu" "*.Mask")
+			(layers "*.Cu" "*.Mask")
 		)
 		(pad "" np_thru_hole circle
@@
 			(size 1.1176 1.1176)
 			(drill 1.1176)
-			(layers "F&B.Cu" "*.Mask")
+			(layers "*.Cu" "*.Mask")
 		)
 		(pad "+" thru_hole oval
@@
 				(font
 					(size 1 1)
-					(thickness 0.1)
+					(thickness 0.15)
 				)
 			)
@@
 			(size 1.1176 1.1176)
 			(drill 1.1176)
-			(layers "F&B.Cu" "*.Mask")
+			(layers "*.Cu" "*.Mask")
 		)
 		(pad "" np_thru_hole circle
@@
 			(size 1.1176 1.1176)
 			(drill 1.1176)
-			(layers "F&B.Cu" "*.Mask")
+			(layers "*.Cu" "*.Mask")
 		)
 		(pad "+" thru_hole oval
@@
 				(font
 					(size 1 1)
-					(thickness 0.1)
+					(thickness 0.15)
 				)
 			)
@@
 			(size 1.1176 1.1176)
 			(drill 1.1176)
-			(layers "F&B.Cu" "*.Mask")
+			(layers "*.Cu" "*.Mask")
 		)
 		(pad "" np_thru_hole circle
@@
 			(size 1.1176 1.1176)
 			(drill 1.1176)
-			(layers "F&B.Cu" "*.Mask")
+			(layers "*.Cu" "*.Mask")
 		)
 		(pad "+" thru_hole oval
@@
 				(font
 					(size 1 1)
-					(thickness 0.1)
+					(thickness 0.15)
 				)
 			)
@@
 			(size 1.1176 1.1176)
 			(drill 1.1176)
-			(layers "F&B.Cu" "*.Mask")
+			(layers "*.Cu" "*.Mask")
 		)
 		(pad "" np_thru_hole circle
@@
 			(size 1.1176 1.1176)
 			(drill 1.1176)
-			(layers "F&B.Cu" "*.Mask")
+			(layers "*.Cu" "*.Mask")
 		)
 		(pad "+" thru_hole oval
@@
 				(font
 					(size 1 1)
-					(thickness 0.1)
+					(thickness 0.15)
 				)
 			)
@@
 			(size 1.1176 1.1176)
 			(drill 1.1176)
-			(layers "F&B.Cu" "*.Mask")
+			(layers "*.Cu" "*.Mask")
 		)
 		(pad "" np_thru_hole circle
@@
 			(size 1.1176 1.1176)
 			(drill 1.1176)
-			(layers "F&B.Cu" "*.Mask")
+			(layers "*.Cu" "*.Mask")
 		)
 		(pad "+" thru_hole oval
@@
 				(font
 					(size 1 1)
-					(thickness 0.1)
+					(thickness 0.15)
 				)
 			)
@@
 			(size 1.1176 1.1176)
 			(drill 1.1176)
-			(layers "F&B.Cu" "*.Mask")
+			(layers "*.Cu" "*.Mask")
 		)
 		(pad "" np_thru_hole circle
@@
 			(size 1.1176 1.1176)
 			(drill 1.1176)
-			(layers "F&B.Cu" "*.Mask")
+			(layers "*.Cu" "*.Mask")
 		)
 		(pad "+" thru_hole oval
@@
 				(font
 					(size 1 1)
-					(thickness 0.1)
+					(thickness 0.15)
 				)
 			)
@@
 			(size 1.1176 1.1176)
 			(drill 1.1176)
-			(layers "F&B.Cu" "*.Mask")
+			(layers "*.Cu" "*.Mask")
 		)
 		(pad "" np_thru_hole circle
@@
 			(size 1.1176 1.1176)
 			(drill 1.1176)
-			(layers "F&B.Cu" "*.Mask")
+			(layers "*.Cu" "*.Mask")
 		)
 		(pad "+" thru_hole oval
@@
 				(font
 					(size 1 1)
-					(thickness 0.1)
+					(thickness 0.15)
 				)
 			)
@@
 			(size 1.1176 1.1176)
 			(drill 1.1176)
-			(layers "F&B.Cu" "*.Mask")
+			(layers "*.Cu" "*.Mask")
 		)
 		(pad "" np_thru_hole circle
@@
 			(size 1.1176 1.1176)
 			(drill 1.1176)
-			(layers "F&B.Cu" "*.Mask")
+			(layers "*.Cu" "*.Mask")
 		)
 		(pad "+" thru_hole oval
@@
 				(font
 					(size 1 1)
-					(thickness 0.1)
+					(thickness 0.15)
 				)
 			)
@@
 			(size 1.1176 1.1176)
 			(drill 1.1176)
-			(layers "F&B.Cu" "*.Mask")
+			(layers "*.Cu" "*.Mask")
 		)
 		(pad "" np_thru_hole circle
@@
 			(size 1.1176 1.1176)
 			(drill 1.1176)
-			(layers "F&B.Cu" "*.Mask")
+			(layers "*.Cu" "*.Mask")
 		)
 		(pad "+" thru_hole oval
@@
 				(font
 					(size 1 1)
-					(thickness 0.1)
+					(thickness 0.15)
 				)
 			)
@@
 				(font
 					(size 1 1)
-					(thickness 0.1)
+					(thickness 0.15)
 				)
 			)
@@
 			(size 1.1176 1.1176)
 			(drill 1.1176)
-			(layers "F&B.Cu" "*.Mask")
+			(layers "*.Cu" "*.Mask")
 		)
 		(pad "" np_thru_hole circle
@@
 			(size 1.1176 1.1176)
 			(drill 1.1176)
-			(layers "F&B.Cu" "*.Mask")
+			(layers "*.Cu" "*.Mask")
 		)
 		(pad "+" thru_hole oval
@@
 				(font
 					(size 1 1)
-					(thickness 0.1)
+					(thickness 0.15)
 				)
 			)
@@
 			(size 1.1176 1.1176)
 			(drill 1.1176)
-			(layers "F&B.Cu" "*.Mask")
+			(layers "*.Cu" "*.Mask")
 		)
 		(pad "" np_thru_hole circle
@@
 			(size 1.1176 1.1176)
 			(drill 1.1176)
-			(layers "F&B.Cu" "*.Mask")
+			(layers "*.Cu" "*.Mask")
 		)
 		(pad "+" thru_hole oval
@@
 				(font
 					(size 1 1)
-					(thickness 0.1)
+					(thickness 0.15)
 				)
 			)
@@
 			(size 1.1176 1.1176)
 			(drill 1.1176)
-			(layers "F&B.Cu" "*.Mask")
+			(layers "*.Cu" "*.Mask")
 		)
 		(pad "" np_thru_hole circle
@@
 			(size 1.1176 1.1176)
 			(drill 1.1176)
-			(layers "F&B.Cu" "*.Mask")
+			(layers "*.Cu" "*.Mask")
 		)
 		(pad "+" thru_hole oval
@@
 				(font
 					(size 1 1)
-					(thickness 0.1)
+					(thickness 0.15)
 				)
 			)
@@
 			(size 1.1176 1.1176)
 			(drill 1.1176)
-			(layers "F&B.Cu" "*.Mask")
+			(layers "*.Cu" "*.Mask")
 		)
 		(pad "" np_thru_hole circle
@@
 			(size 1.1176 1.1176)
 			(drill 1.1176)
-			(layers "F&B.Cu" "*.Mask")
+			(layers "*.Cu" "*.Mask")
 		)
 		(pad "+" thru_hole oval
@@
 			(font
 				(size 1 1)
-				(thickness 0.1)
+				(thickness 0.15)
 			)
 			(justify left bottom)
@@
 			(font
 				(size 1 1)
-				(thickness 0.1)
+				(thickness 0.15)
 			)
 			(justify left bottom)
@@
 			(font
 				(size 1 1)
-				(thickness 0.1)
+				(thickness 0.15)
 			)
 			(justify left bottom)
@@
 			(font
 				(size 1 1)
-				(thickness 0.1)
+				(thickness 0.15)
 			)
 			(justify left bottom)
@@
 			(font
 				(size 1 1)
-				(thickness 0.1)
+				(thickness 0.15)
 			)
 			(justify left bottom)
@@
 			(font
 				(size 1 1)
-				(thickness 0.1)
+				(thickness 0.15)
 			)
 			(justify left bottom)
@@
 			(font
 				(size 1 1)
-				(thickness 0.1)
+				(thickness 0.15)
 			)
 			(justify left bottom)
