File: PCB/Buttons_Flash/Buttons_Flash.kicad_sch (KiCad schematic)
At the start: 20 parts, among them J1 Switches, J2 LEDs, J3 Power, U1 74HC595, U2 74HC595, U3 74HC595, U4 74HC165

Commit message: PCB Buttons Flash
Parts:
- added H1, H2, H3, H4, H5, H6: MountingHole, MountingHole:MountingHole_3.2mm_M3, symbol Mechanical:MountingHole

Commit message: Fader Breakout Board
Other:
- title: (none) -> Flash Buttons Digitast
Changed lines of the file:
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@@
 	(generator_version "8.0")
 	(paper "A4")
+	(title_block
+		(title "Flash Buttons Digitast")
+		(date "2024-09-19")
+		(rev "1")
+	)
 	(junction
 		(at 207.01 140.97)
