File: PCB/Keys_Flash/Keys_Flash.kicad_pcb (KiCad board)
At the start: 2 copper layers, 255 x 68 mm, 86 parts, among them J1 Switches, J2 LEDs, J3 Power, U1 74HC595, U2 74HC595, U3 74HC595, U4 74HC165

Commit message: Keyboard
Routing:
- net GND: vias 95 -> 104
